Commit message: Implement majority of class for constant curvature with working transforms

File: src/prius_description/urdf/prius.urdf (robot description, URDF)
Before this commit: robot prius, 9 links, 8 joints
Links:
- added link imu_link, mass 0.001; collision box size=.001 .001 .001; visual box size=0.001 0.001 0.001
Joints:
- added joint imu_joint: type fixed, parent base_link, child imu_link, origin xyz=0 0 0.19, axis 1 0 0

Commit message: last bugfixes plus rewriting for error ellipses

File: src/prius_description/urdf/prius.urdf (robot description, URDF)
Before this commit: robot prius, 10 links, 9 joints
Joints:
- joint base_link_connection: origin xyz=1.45 0 0 rpy=0 0 1.57 -> xyz=1.45 0 0 rpy=0 0 1.57079632679
